Commit message: Working camera pipeline: horizontal camera orientation, custom world with Sensors plugin and permanent blue box, cleaned xacro, fixed setup.py

File: urdf/camera.xacro (robot description, xacro)
@@ -23,5 +23,5 @@
     <parent link="lbr_link_ee"/>
     <child link="camera_link"/>
-    <origin xyz="0 0 0.02" rpy="0 0 0"/>
+    <origin xyz="0 0 0.02" rpy="0 -1.5708 0"/>
   </joint>
   <gazebo reference="camera_link">
@@ -43,11 +43,5 @@
       <always_on>true</always_on>
       <visualize>true</visualize>
-      <plugin filename="gz-sim-sensors-system" name="gz::sim::systems::Sensors">
-        <render_engine>ogre2</render_engine>
-      </plugin>
     </sensor>
   </gazebo>
-    <plugin filename="gz-sim-sensors-system" name="gz::sim::systems::Sensors">
-      <render_engine>ogre2</render_engine>
-    </plugin>
 </robot>

Commit message: Add face tracking: spawn scanned face model, MediaPipe face detector node, and proportional pan/tilt tracking controller
- db_face model (Scaniverse scan, GLB) spawned via launch at -0.9 0 1.2 with 10deg tilt
- face_detector_node: Face Landmarker (VIDEO mode) publishes nose-tip error on /face_tracking/error + debug image
- face_tracker_controller: P-control on lbr_A1/lbr_A6 with deadband, step cap, joint limits, hold-on-loss
- camera roll fixed 180deg in camera.xacro; blue box removed from world

File: urdf/camera.xacro (robot description, xacro)
@@ -23,5 +23,5 @@
     <parent link="lbr_link_ee"/>
     <child link="camera_link"/>
-    <origin xyz="0 0 0.02" rpy="0 -1.5708 0"/>
+    <origin xyz="0 0 0.02" rpy="3.14159 -1.5708 0"/>
   </joint>
   <gazebo reference="camera_link">

Commit message: Update camera and instrument mount transforms to real hardware measurements (cam: 7.5cm out, 3.1cm right; instrument: 7.5cm out, 7.5cm right) with easy-to-adjust xacro properties

File: urdf/camera.xacro (robot description, xacro)
@@ -1,4 +1,18 @@
 <?xml version="1.0"?>
 <robot xmlns:xacro="http://www.ros.org/wiki/xacro">
+  <!--
+    ============================================================
+    MOUNT CONFIGURATION — change these numbers when mount changes
+    All values in meters, in lbr_link_ee local frame:
+      x = distance out from flange face (toward patient)
+      y = distance right of center (positive = patient sees it left)
+      z = distance up/down from center (0 = in line)
+    rpy = orientation to make camera face -X in world (verified working)
+    ============================================================
+  -->
+  <xacro:property name="cam_x"   value="0.075"/>
+  <xacro:property name="cam_y"   value="0.031"/>
+  <xacro:property name="cam_z"   value="0.0"/>
+  <xacro:property name="cam_rpy" value="3.14159 -1.5708 0"/>
   <link name="camera_link">
     <visual>
@@ -17,5 +31,6 @@
     <inertial>
       <mass value="0.05"/>
-      <inertia ixx="0.0001" ixy="0" ixz="0" iyy="0.0001" iyz="0" izz="0.0001"/>
+      <inertia ixx="0.0001" ixy="0" ixz="0"
+               iyy="0.0001" iyz="0" izz="0.0001"/>
     </inertial>
   </link>
@@ -23,5 +38,5 @@
     <parent link="lbr_link_ee"/>
     <child link="camera_link"/>
-    <origin xyz="0 0 0.02" rpy="3.14159 -1.5708 0"/>
+    <origin xyz="${cam_x} ${cam_y} ${cam_z}" rpy="${cam_rpy}"/>
   </joint>
   <gazebo reference="camera_link">

File: urdf/laser_pointer.xacro (robot description, xacro)
@@ -2,16 +2,24 @@
 <robot xmlns:xacro="http://www.ros.org/wiki/xacro">
   <!--
-    Laser pointer emitter: small black module stacked directly above
-    the camera, as close as physically plausible (1.5cm center-to-center).
-    No beam geometry — the beam is represented by a projected dot
-    (see laser_dot_node), which appears where the laser hits a surface.
+    ============================================================
+    INSTRUMENT MOUNT CONFIGURATION
+    Change these numbers when the instrument position changes.
+    x = distance out from flange face (toward patient)
+    y = distance right of center
+    z = distance up/down from center
+    ============================================================
   -->
+  <xacro:property name="inst_x"   value="0.075"/>
+  <xacro:property name="inst_y"   value="0.075"/>
+  <xacro:property name="inst_z"   value="0.0"/>
+  <xacro:property name="inst_rpy" value="3.14159 -1.5708 0"/>
+  <!-- Instrument body (dermascope placeholder) -->
   <link name="laser_pointer_link">
     <visual>
       <origin xyz="0.01 0 0" rpy="0 1.5708 0"/>
       <geometry>
-        <cylinder radius="0.006" length="0.04"/>
+        <cylinder radius="0.008" length="0.04"/>
       </geometry>
-      <material name="laser_body_black">
+      <material name="instrument_black">
         <color rgba="0.05 0.05 0.05 1"/>
       </material>
@@ -20,7 +28,7 @@
       <origin xyz="0.031 0 0" rpy="0 1.5708 0"/>
       <geometry>
-        <cylinder radius="0.004" length="0.004"/>
+        <cylinder radius="0.005" length="0.005"/>
       </geometry>
-      <material name="laser_aperture_gray">
+      <material name="instrument_gray">
         <color rgba="0.4 0.4 0.4 1"/>
       </material>
@@ -28,5 +36,6 @@
     <inertial>
       <mass value="0.03"/>
-      <inertia ixx="0.00001" ixy="0" ixz="0" iyy="0.00001" iyz="0" izz="0.00001"/>
+      <inertia ixx="0.00001" ixy="0" ixz="0"
+               iyy="0.00001" iyz="0" izz="0.00001"/>
     </inertial>
   </link>
@@ -34,7 +43,5 @@
     <parent link="lbr_link_ee"/>
     <child link="laser_pointer_link"/>
-    <!-- 1.5cm above the camera mount; flip sign of the -0.015 if it
-         renders below the camera instead of above -->
-    <origin xyz="0.015 0 0.02" rpy="3.14159 -1.5708 0"/>
+    <origin xyz="${inst_x} ${inst_y} ${inst_z}" rpy="${inst_rpy}"/>
   </joint>
 </robot>

File: urdf/realsense_camera.xacro (robot description, xacro)
@@ -1,4 +1,18 @@
 <?xml version="1.0"?>
 <robot xmlns:xacro="http://www.ros.org/wiki/xacro">
+  <!--
+    ============================================================
+    MOUNT CONFIGURATION — change these numbers when mount changes
+    All values in meters, in lbr_link_ee local frame:
+      x = distance out from flange face (toward patient)
+      y = distance right of center
+      z = distance up/down from center (0 = in line)
+    rpy = orientation to make camera face -X in world (verified working)
+    ============================================================
+  -->
+  <xacro:property name="cam_x"   value="0.075"/>
+  <xacro:property name="cam_y"   value="0.031"/>
+  <xacro:property name="cam_z"   value="0.0"/>
+  <xacro:property name="cam_rpy" value="3.14159 -1.5708 0"/>
   <link name="realsense_link">
     <visual>
@@ -12,5 +26,6 @@
     <inertial>
       <mass value="0.072"/>
-      <inertia ixx="0.0001" ixy="0" ixz="0" iyy="0.0001" iyz="0" izz="0.0001"/>
+      <inertia ixx="0.0001" ixy="0" ixz="0"
+               iyy="0.0001" iyz="0" izz="0.0001"/>
     </inertial>
   </link>
@@ -18,5 +33,5 @@
     <parent link="lbr_link_ee"/>
     <child link="realsense_link"/>
-    <origin xyz="0 0 0.02" rpy="3.14159 -1.5708 0"/>
+    <origin xyz="${cam_x} ${cam_y} ${cam_z}" rpy="${cam_rpy}"/>
   </joint>
   <gazebo reference="realsense_link">

Commit message: Update camera and instrument mount transforms to real hardware measurements (cam: 7.5cm out, 3.1cm right; instrument: 7.5cm out, 7.5cm right) with easy-to-adjust xacro properties

File: urdf/camera.xacro (robot description, xacro)
@@ -11,7 +11,7 @@
     ============================================================
   -->
-  <xacro:property name="cam_x"   value="0.075"/>
-  <xacro:property name="cam_y"   value="0.031"/>
-  <xacro:property name="cam_z"   value="0.0"/>
+  <xacro:property name="cam_x"   value="0.0"/>
+  <xacro:property name="cam_y"   value="0.0"/>
+  <xacro:property name="cam_z"   value="0.075"/>
   <xacro:property name="cam_rpy" value="3.14159 -1.5708 0"/>
   <link name="camera_link">

File: urdf/laser_pointer.xacro (robot description, xacro)
@@ -10,7 +10,7 @@
     ============================================================
   -->
-  <xacro:property name="inst_x"   value="0.075"/>
-  <xacro:property name="inst_y"   value="0.075"/>
-  <xacro:property name="inst_z"   value="0.0"/>
+  <xacro:property name="inst_x"   value="0.0"/>
+  <xacro:property name="inst_y"   value="0.044"/>
+  <xacro:property name="inst_z"   value="0.075"/>
   <xacro:property name="inst_rpy" value="3.14159 -1.5708 0"/>
   <!-- Instrument body (dermascope placeholder) -->

File: urdf/realsense_camera.xacro (robot description, xacro)
@@ -11,7 +11,7 @@
     ============================================================
   -->
-  <xacro:property name="cam_x"   value="0.075"/>
-  <xacro:property name="cam_y"   value="0.031"/>
-  <xacro:property name="cam_z"   value="0.0"/>
+  <xacro:property name="cam_x"   value="0.0"/>
+  <xacro:property name="cam_y"   value="0.0"/>
+  <xacro:property name="cam_z"   value="0.075"/>
   <xacro:property name="cam_rpy" value="3.14159 -1.5708 0"/>
   <link name="realsense_link">

Commit message: Update camera and instrument mount transforms to match real hardware measurements

File: urdf/camera.xacro (robot description, xacro)
@@ -11,8 +11,8 @@
     ============================================================
   -->
-  <xacro:property name="cam_x"   value="0.0"/>
+  <xacro:property name="cam_x"   value="-0.06465"/>
   <xacro:property name="cam_y"   value="0.0"/>
-  <xacro:property name="cam_z"   value="0.075"/>
-  <xacro:property name="cam_rpy" value="3.14159 -1.5708 0"/>
+  <xacro:property name="cam_z"   value="0.03005"/>
+  <xacro:property name="cam_rpy" value="1.5708 -1.5708 1.5708"/>
   <link name="camera_link">
     <visual>

File: urdf/laser_pointer.xacro (robot description, xacro)
@@ -10,8 +10,8 @@
     ============================================================
   -->
-  <xacro:property name="inst_x"   value="0.0"/>
-  <xacro:property name="inst_y"   value="0.044"/>
-  <xacro:property name="inst_z"   value="0.075"/>
-  <xacro:property name="inst_rpy" value="3.14159 -1.5708 0"/>
+  <xacro:property name="inst_x"   value="-0.0886"/>
+  <xacro:property name="inst_y"   value="0.0"/>
+  <xacro:property name="inst_z"   value="0.0411"/>
+  <xacro:property name="inst_rpy" value="1.5708 -1.5708 1.5708"/>
   <!-- Instrument body (dermascope placeholder) -->
   <link name="laser_pointer_link">

File: urdf/realsense_camera.xacro (robot description, xacro)
@@ -11,8 +11,8 @@
     ============================================================
   -->
-  <xacro:property name="cam_x"   value="0.0"/>
+  <xacro:property name="cam_x"   value="-0.06465"/>
   <xacro:property name="cam_y"   value="0.0"/>
-  <xacro:property name="cam_z"   value="0.075"/>
-  <xacro:property name="cam_rpy" value="3.14159 -1.5708 0"/>
+  <xacro:property name="cam_z"   value="0.03005"/>
+  <xacro:property name="cam_rpy" value="1.5708 -1.5708 1.5708"/>
   <link name="realsense_link">
     <visual>
