Commit message: Add landmark-based raster sweep for real hardware
- raster_sweep_landmark.py: uses MediaPipe forehead landmarks as waypoints
  (36 verified landmark indices across 3 rows, S-pattern)
- raster_sweep_pixel.py: pixel-offset based sweep backup approach
- raster_sweep_hardware.py: world-coordinate backup of original sweep
- landmark_viewer.py: debug tool for identifying landmark indices
- face_detector_node.py: depth mm->meters fix, lbr_link_0 frame, smoothing
- raster_sweep.py: focal length and image size updated for real RealSense
- face_tracker_controller.py: x_bias/y_bias parameters for lens offset
- raster_planner.py: zone coordinates updated for real hardware
- camera_sim.launch.py: READY pose spawn position
- realsense_camera.xacro: real mount transform measurements

File: urdf/realsense_camera.xacro (robot description, xacro)
@@ -12,5 +12,5 @@
   -->
   <xacro:property name="cam_x"   value="-0.06465"/>
-  <xacro:property name="cam_y"   value="0.0"/>
+  <xacro:property name="cam_y"   value="0.0325"/>
   <xacro:property name="cam_z"   value="0.03005"/>
   <xacro:property name="cam_rpy" value="1.5708 -1.5708 1.5708"/>
